Commit message: Added rviz visualization

File: src/legs_description/urdf/legs_feet.urdf (robot description, URDF)
Before this commit: robot bipedal_robot, 10 links, 9 joints
Links:
- link body_link: geometry collision mesh filename=package://legs_description/meshes/final_stl/body_v3_urdf.STL scale=0.001 0.001 0.001; visual mesh filename=package://legs_description/meshes/final_stl/body_v3_urdf.STL scale=0.001 0.001 0.001
- link left_femur_link: geometry collision mesh filename=package://legs_description/meshes/final_stl/femur_L_FINAL.S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 scale=0.001 0.001 0.001; visual mesh filename=package://legs_description/meshes/final_stl/femur_L_FINAL.S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 scale=0.001 0.001 0.001
- link left_foot_link: geometry collision mesh filename=package://legs_description/meshes/final_stl/foot_v4.STL scale=0.001 0.001 0.001; visual mesh filename=package://legs_description/meshes/final_stl/foot_v4.STL scale=0.001 0.001 0.001
- link left_hip_connector_link: geometry collision mesh filename=package://legs_description/meshes/final_stl/hip.STL scale=0.001 0.001 0.001; visual mesh filename=package://legs_description/meshes/final_stl/hip.STL scale=0.001 0.001 0.001
- link left_tibia_link: geometry collision mesh filename=package://legs_description/meshes/final_stl/tibia_final.STL scale=0.001 0.001 0.001; visual mesh filename=package://legs_description/meshes/final_stl/tibia_final.STL scale=0.001 0.001 0.001
- link right_femur_link: geometry collision mesh filename=package://legs_description/meshes/final_stl/femur_R_FINAL.S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 scale=0.001 0.001 0.001; visual mesh filename=package://legs_description/meshes/final_stl/femur_R_FINAL.S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 scale=0.001 0.001 0.001
- link right_foot_link: geometry collision mesh filename=package://legs_description/meshes/final_stl/foot_v4.STL scale=0.001 0.001 0.001; visual mesh filename=package://legs_description/meshes/final_stl/foot_v4.STL scale=0.001 0.001 0.001
- link right_hip_connector_link: geometry collision mesh filename=package://legs_description/meshes/final_stl/hip.STL scale=0.001 0.001 0.001; visual mesh filename=package://legs_description/meshes/final_stl/hip.STL scale=0.001 0.001 0.001
- link right_tibia_link: geometry collision mesh filename=package://legs_description/meshes/final_stl/tibia_final.STL scale=0.001 0.001 0.001; visual mesh filename=package://legs_description/meshes/final_stl/tibia_final.STL scale=0.001 0.001 0.001
